File: PneumaticsControlBoard/Pneumatics Control Unit V1.kicad_pcb (KiCad board)
At the start: 2 copper layers, 53.6 x 65.4 mm, 78 parts, among them J1 TX_PORT, J10 Conn_01x02_Male, J11 Conn_01x02_Male, J12 10118194-0001LF, J2 RX_PORT, J3 MICROMOD-2222, J4 Conn_01x02_Male, J5 Conn_01x02_Male, J6 Conn_01x02_Male, J7 Conn_01x02_Male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

Commit message: Add files via upload
Parts:
- added J13: Conn_01x03_Male, Header:Conn_1x3, F.Cu at (108.3, 117.6)
- added J14: Conn_01x03_Male, Header:Conn_1x3, F.Cu at (145.2, 108.1)
- moved C24 0.05 mm to (114.8, 99.4)
- moved C25 0.05 mm to (110.2, 99.4)
Connections:
- net 3.3V renamed /220uF
- C10 pad 1: USB_V -> Net-(C10-Pad1)
- C23 pad 1: 5V_R -> Net-(U3-OUTPUT)
- C25 pad 1: 5V_L -> Net-(U4-OUTPUT)
- C5 pad 1: USB_V -> Net-(C10-Pad1)
- C8 pad 1: USB_V -> Net-(C10-Pad1)
- C9 pad 1: USB_V -> Net-(C10-Pad1)
- J10 pad 2: 5V_R -> /solenoid_power_2
- J11 pad 2: 5V_R -> /solenoid_power_2
- J12 pad 1: USB_V -> Net-(J12-Pad1)
- J3 pad 9: USB_V -> Net-(J3-USB_VIN)
- J4 pad 2: 5V_L -> /solenoid_power
- J5 pad 2: 5V_L -> /solenoid_power
- J6 pad 2: 5V_L -> /solenoid_power
- J7 pad 2: 5V_R -> /solenoid_power_2
- J8 pad 2: 5V_L -> /solenoid_power
- J9 pad 2: 5V_R -> /solenoid_power_2
- U3 pad 3: 5V_R -> Net-(U3-OUTPUT)
- U4 pad 3: 5V_L -> Net-(U4-OUTPUT)
Routing:
- net /RS485_B_12V: track 45.0 -> 113.0 mm
- net 5V_R: track 66.5 -> 0.00 mm, vias 2 -> 0
- net USB_V: track 65.2 -> 0.00 mm, vias 3 -> 0
- net Net-(C10-Pad1): track 0.00 -> 65.2 mm, vias 0 -> 3
- net /solenoid_power_2: track 0.00 -> 55.6 mm
- net /solenoid_power: track 0.00 -> 52.2 mm
- net 5V_L: track 50.3 -> 0.00 mm
- net Net-(U4-OUTPUT): track 0.00 -> 17.9 mm
- net Net-(U3-OUTPUT): track 0.00 -> 16.7 mm, vias 0 -> 1
- net GND: vias 28 -> 34
- added copper zone on In1.Cu, net (none)
- added copper zone on In2.Cu, net (none)
Other:
- copper layers 2 -> 4

Commit message: Add files via upload
Routing:
- net GND: track 36.9 -> 47.2 mm, vias 34 -> 38
Changed lines of the file:
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@@
     (grid_origin 191.516 98.552)
     (pcbplotparams
-      (layerselection 0x00010f0_ffffffff)
+      (layerselection 0x00010fc_ffffffff)
       (plot_on_all_layers_selection 0x0000000_00000000)
       (disableapertmacros false)
       (usegerberextensions true)
-      (usegerberattributes true)
-      (usegerberadvancedattributes true)
-      (creategerberjobfile true)
+      (usegerberattributes false)
+      (usegerberadvancedattributes false)
+      (creategerberjobfile false)
       (dashed_line_dash_ratio 12.000000)
       (dashed_line_gap_ratio 3.000000)
@@
     (property "ki_keywords" "cap capacitor")
     (attr smd)
-    (fp_text reference "C25" (at 0 -1.68 90) (layer "F.SilkS")
+    (fp_text reference "C25" (at 0 -1.397 90) (layer "F.SilkS")
         (effects (font (size 1 1) (thickness 0.15)))
     )
@@
       (stroke (width 0.1) (type solid)) (fill none) (layer "F.Fab"))
     (pad "1" smd rect locked (at -1.3 -2.7) (size 0.4 1.35) (layers "F.Cu" "F.Paste" "F.Mask")
-      (net 78 "Net-(J12-Pad1)") (pinfunction "1") (pintype "passive"))
+      (net 78 "Net-(J12-Pad1)") (pinfunction "1") (pintype "passive") (clearance 0.2))
     (pad "2" smd rect locked (at -0.65 -2.7) (size 0.4 1.35) (layers "F.Cu" "F.Paste" "F.Mask")
       (net 76 "Net-(J12-Pad2)") (pinfunction "2") (pintype "passive"))
@@
   (segment (start 115.808 120.61) (end 115.808 118.364) (width 0.25) (layer "B.Cu") (net 1))
   (segment (start 115.401489 121.016511) (end 115.401489 124.672489) (width 0.25) (layer "B.Cu") (net 1))
+  (segment (start 131.572 118.11) (end 129.413 118.11) (width 0.35) (layer "F.Cu") (net 2))
   (segment (start 130.81 91.6178) (end 129.54 91.6178) (width 0.35) (layer "F.Cu") (net 2))
   (segment (start 145.685 129.413) (end 143.185 129.413) (width 0.35) (layer "F.Cu") (net 2))
-  (segment (start 132.461 98.256) (end 132.6515 98.0655) (width 0.35) (layer "F.Cu") (net 2))
   (segment (start 130.81 82.1182) (end 132.08 82.1182) (width 0.35) (layer "F.Cu") (net 2))
   (segment (start 132.6515 98.0655) (end 135.154 98.0655) (width 0.35) (layer "F.Cu") (net 2))
+  (segment (start 122.682 103.378) (end 120.523 103.378) (width 0.35) (layer "F.Cu") (net 2))
   (segment (start 121.666 94.7667) (end 121.4755 94.5762) (width 0.35) (layer "F.Cu") (net 2))
   (segment (start 130.81 82.1182) (end 129.54 82.1182) (width 0.35) (layer "F.Cu") (net 2))
-  (segment (start 129.0073 99.2364) (end 129.0955 99.1482) (width 0.35) (layer "F.Cu") (net 2))
   (segment (start 128.27 91.6178) (end 129.54 91.6178) (width 0.35) (layer "F.Cu") (net 2))
-  (segment (start 118.4275 99.1482) (end 119.0378 99.1482) (width 0.35) (layer "F.Cu") (net 2))
   (segment (start 135.154 98.0655) (end 135.1915 98.028) (width 0.35) (layer "F.Cu") (net 2))
+  (segment (start 132.842 116.84) (end 131.572 118.11) (width 0.35) (layer "F.Cu") (net 2))
   (segment (start 124.0155 94.7667) (end 121.666 94.7667) (width 0.35) (layer "F.Cu") (net 2))
+  (segment (start 120.523 103.378) (end 118.364 105.537) (width 0.35) (layer "F.Cu") (net 2))
   (segment (start 132.08 91.6178) (end 130.81 91.6178) (width 0.35) (layer "F.Cu") (net 2))
   (segment (start 129.54 82.1182) (end 128.27 82.1182) (width 0.35) (layer "F.Cu") (net 2))
@@
   (via (at 129.286 87.63) (size 0.8) (drill 0.4) (layers "F.Cu" "B.Cu") (net 2))
   (via (at 118.364 105.537) (size 0.8) (drill 0.4) (layers "F.Cu" "B.Cu") (free) (net 2))
+  (via (at 122.682 103.378) (size 0.8) (drill 0.4) (layers "F.Cu" "B.Cu") (free) (net 2))
   (via (at 144.78 78.613) (size 0.8) (drill 0.4) (layers "F.Cu" "B.Cu") (free) (net 2))
   (via (at 149.225 105.537) (size 0.8) (drill 0.4) (layers "F.Cu" "B.Cu") (free) (net 2))
@@
   (via (at 134.747 108.458) (size 0.8) (drill 0.4) (layers "F.Cu" "B.Cu") (free) (net 2))
   (via (at 132.08 87.249) (size 0.8) (drill 0.4) (layers "F.Cu" "B.Cu") (free) (net 2))
+  (via (at 129.413 118.11) (size 0.8) (drill 0.4) (layers "F.Cu" "B.Cu") (free) (net 2))
   (via (at 129.921 102.87) (size 0.8) (drill 0.4) (layers "F.Cu" "B.Cu") (free) (net 2))
   (via (at 130.937 114.0085) (size 0.8) (drill 0.4) (layers "F.Cu" "B.Cu") (net 2))
+  (via (at 117.221 90.805) (size 0.8) (drill 0.4) (layers "F.Cu" "B.Cu") (free) (net 2))
   (via (at 149.098 100.203) (size 0.8) (drill 0.4) (layers "F.Cu" "B.Cu") (net 2))
   (via (at 148.336 124.079) (size 0.8) (drill 0.4) (layers "F.Cu" "B.Cu") (free) (net 2))
@@
   (via (at 132.588 127.254) (size 0.8) (drill 0.4) (layers "F.Cu" "B.Cu") (free) (net 2))
   (via (at 117.475 110.744) (size 0.8) (drill 0.4) (layers "F.Cu" "B.Cu") (free) (net 2))
+  (via (at 119.888 90.043) (size 0.8) (drill 0.4) (layers "F.Cu" "B.Cu") (free) (net 2))
   (via (at 132.588 93.98) (size 0.8) (drill 0.4) (layers "F.Cu" "B.Cu") (free) (net 2))
   (via (at 135.128 102.87) (size 0.8) (drill 0.4) (layers "F.Cu" "B.Cu") (free) (net 2))
@@
   (segment (start 129.4755 87.8195) (end 129.4755 89.50625) (width 0.25) (layer "B.Cu") (net 2))
   (segment (start 131.191 99.187) (end 130.2255 98.2215) (width 0.2) (layer "B.Cu") (net 2))
-  (segment (start 109.407 90.878498) (end 109.332001 90.803499) (width 0.35) (layer "B.Cu") (net 2))
   (segment (start 128.7255 98.080272) (end 128.866728 98.2215) (width 0.2) (layer "B.Cu") (net 2))
   (segment (start 120.015 98.465772) (end 120.7255 97.755272) (width 0.2) (layer "B.Cu") (net 2))
@@
   (segment (start 122.016739 95.981739) (end 122.2255 96.1905) (width 0.2) (layer "B.Cu") (net 2))
   (segment (start 120.7255 97.755272) (end 120.7255 97.05625) (width 0.2) (layer "B.Cu") (net 2))
-  (segment (start 109.586001 112.647499) (end 109.586001 112.990199) (width 0.35) (layer "B.Cu") (net 2))
   (segment (start 128.866728 98.2215) (end 130.2255 98.2215) (width 0.2) (layer "B.Cu") (net 2))
-  (segment (start 109.407 79.2985) (end 109.459001 79.246499) (width 0.35) (layer "B.Cu") (net 2))
   (segment (start 131.7255 98.1975) (end 131.7255 97.05625) (width 0.2) (layer "B.Cu") (net 2))
-  (segment (start 109.332001 91.171001) (end 109.332001 90.803499) (width 0.35) (layer "B.Cu") (net 2))
+  (segment (start 119.888 90.043) (end 117.983 90.043) (width 0.35) (layer "B.Cu") (net 2))
   (segment (start 120.015 99.06) (end 120.015 98.465772) (width 0.2) (layer "B.Cu") (net 2))
   (segment (start 139.250011 95.816011) (end 139.250011 97.05625) (width 0.35) (layer "B.Cu") (net 2))
   (segment (start 130.2255 98.2215) (end 130.2255 97.05625) (width 0.2) (layer "B.Cu") (net 2))
+  (segment (start 117.983 90.043) (end 117.221 90.805) (width 0.35) (layer "B.Cu") (net 2))
   (segment (start 131.191 99.187) (end 131.191 98.732) (width 0.2) (layer "B.Cu") (net 2))
   (segment (start 121.031 120.8825) (end 119.9935 121.92) (width 0.35) (layer "B.Cu") (net 2))
@@
   (segment (start 128.524 107.188) (end 128.524 102.743) (width 0.25) (layer "F.Cu") (net 23))
   (segment (start 139.954 107.696) (end 139.446 107.188) (width 0.25) (layer "F.Cu") (net 23))
-  (segment (start 128.27 102.489) (end 121.026 102.489) (width 0.25) (layer "F.Cu") (net 23))
-  (segment (start 139.446 107.188) (end 128.524 107.188) (width 0.25) (layer "F.Cu") (net 23))
-  (segment (start 128.524 102.743) (end 128.27 102.489) (width 0.25) (layer "F.Cu") (net 23))
+  (segment (start 128.524 102.743) (end 127.889 102.108) (width 0.25) (layer "F.Cu") (net 23))
   (segment (start 139.954 115.697) (end 139.954 107.696) (width 0.25) (layer "F.Cu") (net 23))
+  (segment (start 139.446 107.188) (end 128.524 107.188) (width 0.25) (layer "F.Cu") (net 23))
+  (segment (start 121.407 102.108) (end 121.026 102.489) (width 0.25) (layer "F.Cu") (net 23))
+  (segment (start 127.889 102.108) (end 121.407 102.108) (width 0.25) (layer "F.Cu") (net 23))
   (via (at 121.026 102.489) (size 0.8) (drill 0.4) (layers "F.Cu" "B.Cu") (net 23))
   (segment (start 121.2255 97.05625) (end 121.2255 102.2895) (width 0.2) (layer "B.Cu") (net 23))
@@
   (segment (start 116.326 122.152) (end 116.326 124.979457) (width 0.25) (layer "F.Cu") (net 66))
   (segment (start 116.326 122.152) (end 108.861 122.152) (width 0.25) (layer "F.Cu") (net 66))
-  (segment (start 114.812 100.4825) (end 114.808 100.4785) (width 0.25) (layer "F.Cu") (net 66))
   (segment (start 130.937 112.014) (end 132.5753 110.3757) (width 0.25) (layer "F.Cu") (net 66))
   (segment (start 122.9855 114.4765) (end 123.5215 114.4765) (width 0.25) (layer "F.Cu") (net 66))
@@
   (segment (start 141.53952 128.20848) (end 150.42952 128.20848) (width 0.25) (layer "F.Cu") (net 66))
   (segment (start 148.336 113.157) (end 145.161 113.157) (width 0.25) (layer "F.Cu") (net 66))
-  (segment (start 114.812 100.5333) (end 114.808 100.5293) (width 0.25) (layer "F.Cu") (net 66))
   (segment (start 126.39048 113.865684) (end 126.39048 112.11552) (width 0.25) (layer "F.Cu") (net 66))
   (segment (start 108.861 122.152) (end 108.331 122.682) (width 0.25) (layer "F.Cu") (net 66))
@@
   (segment (start 136.906 102.997) (end 140.081 102.997) (width 0.25) (layer "B.Cu") (net 87))
   (segment (start 140.081 102.997) (end 145.161 108.077) (width 0.25) (layer "B.Cu") (net 87))
-  (segment (start 110.232 100.4825) (end 110.236 100.4785) (width 0.25) (layer "F.Cu") (net 88))
   (segment (start 108.331 106.6125) (end 108.331 117.602) (width 0.25) (layer "F.Cu") (net 88))
   (segment (start 110.232 104.7115) (end 108.331 106.6125) (width 0.25) (layer "F.Cu") (net 88))
   (segment (start 110.232 104.7115) (end 110.232 100.4825) (width 0.25) (layer "F.Cu") (net 88))
-  (segment (start 110.232 100.5333) (end 110.236 100.5293) (width 0.25) (layer "F.Cu") (net 88))
   (zone (net 2) (net_name "GND") (layers F&B.Cu) (hatch edge 0.508)
     (connect_pads (clearance 0.508))
