File: PneumaticsControlBoard/Pneumatics Control Unit V1.kicad_sch (KiCad schematic)
At the start: 78 parts

Commit message: Add files via upload
Other:
- note added: "5V rail (500mA)x2 ------------- Pneumatics ~800mA ------------- Total ~800mA"
- note removed: "5V rail (500mA) ------------- Pneumatics ~ ------------- Total ~"
